Commit message: customised lidar, inflation radius and epmc params

File: mobo_bot_description/urdf/four_wheel_base/ros2_control.xacro (robot description, xacro)
@@ -13,6 +13,6 @@
       <joint name="front_left_wheel_joint">
         <command_interface name="velocity">
-            <param name="min">-15.0</param>
-            <param name="max">15.0</param>
+            <param name="min">-10.0</param>
+            <param name="max">10.0</param>
         </command_interface>
         <state_interface name="position"/>
@@ -21,6 +21,6 @@
       <joint name="front_right_wheel_joint">
         <command_interface name="velocity">
-            <param name="min">-15.0</param>
-            <param name="max">15.0</param>
+            <param name="min">-10.0</param>
+            <param name="max">10.0</param>
         </command_interface>
         <state_interface name="position"/>
@@ -29,6 +29,6 @@
       <joint name="rear_left_wheel_joint">
         <command_interface name="velocity">
-            <param name="min">-15.0</param>
-            <param name="max">15.0</param>
+            <param name="min">-10.0</param>
+            <param name="max">10.0</param>
         </command_interface>
         <state_interface name="position"/>
@@ -37,6 +37,6 @@
       <joint name="rear_right_wheel_joint">
         <command_interface name="velocity">
-            <param name="min">-15.0</param>
-            <param name="max">15.0</param>
+            <param name="min">-10.0</param>
+            <param name="max">10.0</param>
         </command_interface>
         <state_interface name="position"/>

File: mobo_bot_description/urdf/urdf_models/lidar.xacro (robot description, xacro)
@@ -5,9 +5,9 @@
             <parent link="${parent_name}"/>
             <child link="${base_name}"/>
-            <origin xyz="${x} ${y} ${z}" rpy="0 0 0"/>
+            <origin xyz="${x} ${y} ${z}" rpy="0 0 ${pi}"/>  <!-- change yaw to 0 for simulation -->
         </joint>
         <link name="${base_name}">
             <visual>
-                <origin xyz="0 0 -0.02"/>
+                <origin xyz="0 0 -0.02" rpy="0 0 0"/>
                 <geometry>
                     <cylinder radius="0.03" length="0.04"/>
@@ -18,5 +18,5 @@
             </visual>
             <collision>
-                <origin xyz="0 0 -0.02"/>
+                <origin xyz="0 0 -0.02" rpy="0 0 0"/>
                 <geometry>
                     <cylinder radius="0.03" length="0.04"/>
