Commit message: modified imu and camera positions

File: mobo_bot_description/urdf/four_wheel_base/robot.xacro (robot description, xacro)
@@ -129,8 +129,9 @@
         x="0.05" y="0" z="${chassis_height+lidar_z_offset}"
         mass="0.1"/>
+    <xacro:property name="imu_height" value="0.02"/>
     <joint name="imu_joint" type="fixed">
         <parent link="chassis"/>
         <child link="imu"/>
-        <origin xyz="0 0 ${slab_height}"/>
+        <origin xyz="0.075 0 ${slab_height+imu_height}"/>
     </joint>
     <link name="imu"></link>
@@ -143,5 +144,5 @@
         base_name="camera"
         parent_name="chassis"
-        x="0.13" y="0" z="${chassis_height+0.015}"
+        x="0.11" y="0" z="${chassis_height+0.015}"
         mass="0.005" tilt_angle="0.00"/>
 </robot>

Commit message: description chn=anges

File: mobo_bot_description/urdf/four_wheel_base/robot.xacro (robot description, xacro)
@@ -123,5 +123,6 @@
         thickness="${wheel_width}"
         spoke_width="0.005"/>
-    <xacro:property name="lidar_z_offset" value="0.04"/>
+        <!-- Z value determins the height of the laser scans -->
+    <xacro:property name="lidar_z_offset" value="0.03"/>
     <xacro:insert_lidar
         base_name="lidar"

File: mobo_bot_description/urdf/urdf_models/lidar.xacro (robot description, xacro)
@@ -9,5 +9,5 @@
         <link name="${base_name}">
             <visual>
-                <origin xyz="0 0 -0.02"/>
+                <origin xyz="0 0 -0.01"/>
                 <geometry>
                     <cylinder radius="0.03" length="0.04"/>
@@ -18,5 +18,5 @@
             </visual>
             <collision>
-                <origin xyz="0 0 -0.02"/>
+                <origin xyz="0 0 -0.01"/>
                 <geometry>
                     <cylinder radius="0.03" length="0.04"/>
@@ -24,5 +24,5 @@
             </collision>
             <xacro:inertial_cylinder mass="${mass}" length="0.04" radius="0.03">
-                <origin xyz="0 0 -0.02" rpy="0 0 0"/>
+                <origin xyz="0 0 -0.01" rpy="0 0 0"/>
             </xacro:inertial_cylinder>
         </link>
