Commit message: added keepout,speed,docking server + final augmentor script

File: mobo_bot_description/urdf/urdf_models/lidar.xacro (robot description, xacro)
@@ -5,5 +5,5 @@
             <parent link="${parent_name}"/>
             <child link="${base_name}"/>
-            <origin xyz="${x} ${y} ${z}" rpy="0 0 ${pi}"/>  <!-- change yaw to 0 for simulation -->
+            <origin xyz="${x} ${y} ${z}" rpy="0 0 0"/>  <!-- change yaw to 0 for simulation -->
         </joint>
         <link name="${base_name}">
